File: final_project_pcb/final_project_pcb.kicad_sch (KiCad schematic)
At the start: 4 parts, among them U3 Pulse_Sensor

Commit message: lab5_power_estimate
Parts:
- removed U2: ~, symbol Techin514_final_project:MPU6050
- removed U3: Pulse_Sensor, symbol Techin514_final_project:Pulse_Sensor
- added Brd1: SSD1306, SS1306:128x64OLED, symbol SSD1306:SSD1306
- added D1: LED, LED_SMD:LED_0805_2012Metric_Pad1.15x1.40mm_HandSolder, symbol Device:LED
- added M1: Stepper_Motor_bipolar, Stepper_Motor_X27:x27_stepper, symbol Motor:Stepper_Motor_bipolar
- added R2: R, Resistor_SMD:R_0805_2012Metric_Pad1.20x1.40mm_HandSolder, symbol Device:R
- added SW1: SW_Push, symbol Switch:SW_Push
- U1: footprint (none) -> XIAO ESP32S3:XIAO_ESP32_SENSE
Connections:
- net GND: now also Brd1.1 (GND), R2.1
- net at U1.5 (GPIO4_A3_D3_SDA): now also Brd1.4 (SDA)
- net at U1.6 (GPIO6_A5_D5_SCL): now also Brd1.3 (SCL)
- net at U1.1 (GPIO1_A0_D0): now also M1.1
- net at U1.2 (GPIO2_A1_D1): now also M1.2 (-)
- net at U1.3 (GPIO3_A2_D2): now also M1.3
- net at U1.4 (GPIO4_A3_D3): now also M1.4
- net VCC: now reaches U1.8 (5V)
- net VCC: now also Brd1.2 (VCC), SW1.1
- new net: D1.1 (K), R2.2
- new net: D1.2 (A), SW1.2
Other:
- moved on the sheet: BT1, U1
